Commit message: Trying to redo the ikfast for an atlas with proper joint limits, not quite working...

File: adept/adept_common/urdf/OCS_urdf/adept.urdf (robot description, URDF)
Before this commit: robot ADEPT_VIPER_S650, 22 links, 21 joints
Links:
- removed link Adept_Viper_650_Interface_Plate
- added link l_hand, mass 1; collision mesh filename=package://adept_common/meshes/collision/STL/binary/Adept_Vi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; visual mesh filename=package://adept_common/meshes/visual/STL/binary/Adept_Viper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
Joints:
- joint joint_6: child Adept_Viper_650_Interface_Plate -> l_hand
- joint joint_7: parent Adept_Viper_650_Interface_Plate -> l_hand
